File: AmpClassD_Daugher.kicad_pcb (KiCad board)
At the start: 2 copper layers, 67 parts, among them J1 POWER, J10 MONO, J11 LEFT, J2 POWER, J3 AUDIO_IN, J4 ST/MN, J5 GAIN_DEFAULT, J6 SYNC_DEFAULT, J7 MN, J8 MN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

Commit message: schematic updates
Parts:
- added D2: M7, Diode_SMD:D_SMA, F.Cu at (32.0, 55.5)
- added J12: INS, Connector_PinHeader_2.54mm:PinHeader_1x14_P2.54mm_Vertical, F.Cu at (158.1, 48.6)
- added J13: OUTS, Connector_PinHeader_2.54mm:PinHeader_1x14_P2.54mm_Vertical, F.Cu at (162.7, 48.6)
- added J14: PLIM_DEF, Connector_PinHeader_2.54mm:PinHeader_1x02_P2.54mm_Vertical_SMD_Pin1Right, F.Cu at (40.0, 56.8)
- added Q5: MMBT3904, Package_TO_SOT_SMD:SOT-23, F.Cu at (30.2, 60.1)
- added R17: 100k, Resistor_SMD:R_0603_1608Metric_Pad1.05x0.95mm_HandSolder_SmallRef, F.Cu at (34.6, 61.7)
- J5: value GAIN_DEFAULT -> GAIN_DEF
- RV1, RV2: value 2.2k -> 20k
Connections:
- J1 pad 2: +24V -> VCC
- J2 pad 1: +24V -> VCC
- R7 pad 2: (no net) -> MUTE
- U3 pad 6: GVDD -> PLIM

Commit message: layout progress
Parts:
- added J15: PWR, HammerheadAudio:M3_Plated, F.Cu at (120.4, 9.61)
- added J16: GND, HammerheadAudio:M3_Plated, F.Cu at (120.4, 16.3)
- added J17: R+, HammerheadAudio:M3_Plated, F.Cu at (140.0, 40.0)
- added J18: L+, HammerheadAudio:M3_Plated, F.Cu at (140.0, 90.0)
- added JP1: PWR, Jumper:SolderJumper-2_P1.3mm_Open_Pad1.0x1.5mm, F.Cu at (132.6, 8.03)
- added JP2: GND, Jumper:SolderJumper-2_P1.3mm_Open_Pad1.0x1.5mm, F.Cu at (136.9, 8.03)
- added JP3: R+, Jumper:SolderJumper-2_P1.3mm_Open_Pad1.0x1.5mm, F.Cu at (130.0, 40.0)
- added JP4: L+, Jumper:SolderJumper-2_P1.3mm_Open_Pad1.0x1.5mm, F.Cu at (130.0, 90.0)
- J1, J10, J11, J9: footprint HammerheadAudio:Phoenix_Stacked_Marking2_Wider_NoRef -> HammerheadAudio:Phoenix_Stacked_Marking2_Wider_NoRef_Centered
- moved J12 150.3 mm to (8.00, 56.0)
- moved C26 82.1 mm to (46.8, 86.5)
- moved R8 76.7 mm to (51.2, 42.2), turned to 90 degrees
- moved R13 74.2 mm to (54.8, 42.2), turned to 270 degrees
- moved R16 72.2 mm to (71.2, 34.2), turned to 270 degrees
- moved C9 67.4 mm to (48.2, 68.0)
- moved J3 52.5 mm to (7.00, 35.0)
- moved R15 45.9 mm to (73.0, 81.5), turned to 180 degrees
- moved Q5 43.7 mm to (68.8, 39.5)
- moved R17 43.0 mm to (67.8, 34.2), turned to 90 degrees
- moved C8 42.0 mm to (78.8, 54.5), turned to 180 degrees
- moved C15 38.1 mm to (118.2, 65.5), turned to 180 degrees
- moved C16 37.5 mm to (118.2, 63.8)
- moved J14 36.4 mm to (76.0, 62.2), turned to 180 degrees
- moved C10 33.6 mm to (76.5, 81.5)
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Connections:
- J13 pad 2: R- -> R+
- J13 pad 3: R- -> R+
- J13 pad 4: R- -> R+
- J13 pad 5: R+ -> R-
- J13 pad 6: R+ -> R-
- J13 pad 7: R+ -> R-
Other:
- board text added: "|"
- board text added: "| L+/M-"
- board text added: "| L-"
- board text added: "| R+/M+"
- board text added: "| R-"

Commit message: layout progress
Parts:
- moved J16 3.43 mm to (120.4, 19.8)
- renumbered J14 to J12, J12 to J14
Changed lines of the file:
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@@
     (tags "Surface mounted pin header SMD 1x02 2.54mm single row style2 pin1 right")
     (attr smd)
-    (fp_text reference J14 (at 2.25 1.25 90) (layer F.SilkS)
+    (fp_text reference J12 (at 2.25 1.25 90) (layer F.SilkS)
       (effects (font (size 1 1) (thickness 0.15)))
     )
@@
     (descr "Through hole straight pin header, 1x14, 2.54mm pitch, single row")
     (tags "Through hole pin header THT 1x14 2.54mm single row")
-    (fp_text reference J12 (at 0 -2.33) (layer F.SilkS)
+    (fp_text reference J14 (at 0 -2.33) (layer F.SilkS) hide
       (effects (font (size 1 1) (thickness 0.15)))
     )
@@
     (descr "Through hole straight pin header, 1x14, 2.54mm pitch, single row")
     (tags "Through hole pin header THT 1x14 2.54mm single row")
-    (fp_text reference J13 (at 0 -2.33) (layer F.SilkS)
+    (fp_text reference J13 (at 0 -2.33) (layer F.SilkS) hide
       (effects (font (size 1 1) (thickness 0.15)))
     )
@@
   )
   (module HammerheadAudio:M3_Plated (layer F.Cu)
-    (at 120.357501 16.317501)
+    (at 120.357501 19.75)
     (descr "STANDOFF (#4 SCREW)")
     (tags "STANDOFF (#4 SCREW)")

Commit message: layout progress
Parts:
- moved J16 86.4 mm to (70.0, 90.0)
- moved J3 77.7 mm to (72.0, 77.5), turned to 0 degrees
- moved J14 73.6 mm to (81.2, 48.5)
- moved J15 58.8 mm to (70.0, 40.0)
- moved C1 58.3 mm to (90.5, 55.0), turned to 180 degrees
- moved C2 58.2 mm to (90.5, 71.8), turned to 180 degrees
- moved R1 56.0 mm to (90.5, 56.8), turned to 0 degrees
- moved R2 55.9 mm to (90.5, 73.5), turned to 0 degrees
- moved J2 55.8 mm to (65.0, 52.5), turned to 90 degrees
- moved RV1 53.5 mm to (89.8, 68.2), turned to 180 degrees
- moved RV2 53.5 mm to (89.8, 85.0), turned to 180 degrees
- moved R11 50.7 mm to (102.8, 32.2)
- moved R13 50.7 mm to (104.5, 32.2)
- moved Q2 50.7 mm to (100.0, 38.0)
- moved Q4 50.7 mm to (103.8, 38.0)
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Connections:
- J3 pad R: (no net) -> RIN
- J3 pad S: (no net) -> GND
- J3 pad T: (no net) -> LIN
- J4 pad 1: Net-(C6-Pad1) -> Net-(C5-Pad1)
- J4 pad 2: Net-(C5-Pad1) -> Net-(C6-Pad1)
- J4 pad 3: LIN- -> LIN+
- J4 pad 4: LIN+ -> LIN-
Routing:
- net R+: track 0.00 -> 121.1 mm
- net L+: track 0.00 -> 114.3 mm
- net R-: track 0.00 -> 98.7 mm
- net L-: track 0.00 -> 51.1 mm
- net Net-(C15-Pad1): track 0.00 -> 48.3 mm
- net Net-(C17-Pad2): track 0.00 -> 39.3 mm
- net Net-(C16-Pad2): track 0.00 -> 36.5 mm
- net Net-(C14-Pad1): track 0.00 -> 34.8 mm
- net Net-(C16-Pad1): track 0.00 -> 23.5 mm
- net VCC: track 0.00 -> 17.1 mm
- net Net-(C17-Pad1): track 0.00 -> 11.2 mm
- net Net-(C14-Pad2): track 0.00 -> 7.45 mm
- net Net-(J18-Pad1): track 0.00 -> 5.45 mm
- net Net-(J17-Pad1): track 0.00 -> 5.45 mm
- net Net-(C15-Pad2): track 0.00 -> 4.30 mm
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Other:
- board text added: "GAIN DEFAULT"
- board text added: "MONO"
- board text added: "PLIM DEFAULT"
- board text added: "RIGHT"
- board text added: "STEREO"
- board text added: "STEREO VS MONO"
- board text added: "SYNC DEFAULT"
- board text added: "| L- | L+ | R- | R+ |"
- board text removed: "|"
- board text removed: "| L+/M-"
- board text removed: "| L-"
- board text removed: "| R+/M+"
- board text removed: "| R-"

Commit message: initial layout finished
Parts:
- moved JP2 101.3 mm to (77.5, 90.0)
- moved JP1 63.7 mm to (77.5, 40.0)
- moved D2 58.6 mm to (83.5, 43.8)
- moved R13 55.5 mm to (88.0, 85.2)
- moved R7 54.9 mm to (84.5, 85.2)
- moved R8 54.9 mm to (86.2, 85.2)
- moved R11 54.6 mm to (89.8, 85.2)
- moved Q4 48.6 mm to (92.5, 85.2), turned to 180 degrees
- moved Q2 47.4 mm to (96.2, 85.2), turned to 180 degrees
- moved D1 26.4 mm to (92.2, 43.8), turned to 180 degrees
- moved Q3 18.4 mm to (103.0, 46.2), turned to 180 degrees
- moved Q1 18.2 mm to (99.2, 46.2), turned to 180 degrees
- moved R12 16.4 mm to (101.2, 52.2), turned to 90 degrees
- moved R14 16.4 mm to (104.8, 52.2), turned to 90 degrees
- moved R16 16.4 mm to (103.0, 52.2)
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Routing:
- net VCC: track 17.1 -> 317.9 mm, vias 0 -> 2
- net GND: track 2.98 -> 71.4 mm, vias 0 -> 145
- net LIN: track 0.00 -> 46.1 mm
- net SYNC: track 0.00 -> 44.0 mm
- net PLIM: track 0.00 -> 37.7 mm, vias 0 -> 1
- net GVDD: track 0.00 -> 37.4 mm, vias 0 -> 1
- net RIN: track 0.00 -> 35.8 mm
- net Net-(Q4-Pad3): track 0.00 -> 35.6 mm
- net FAULT: track 0.00 -> 34.8 mm, vias 0 -> 1
- net GAIN: track 0.00 -> 30.7 mm, vias 0 -> 1
- net RIN-: track 0.00 -> 21.5 mm
- net L+: track 114.3 -> 133.7 mm
- net RIN+: track 0.00 -> 19.3 mm
- net LIN+: track 0.00 -> 17.8 mm
- net Net-(C6-Pad1): track 0.00 -> 17.1 mm
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- added copper zone on B.Cu, net GND
- added copper zone on F.Cu, net GND
Other:
- board outline added: 80 x 60 mm
- board text added: "FAULT"
- board text added: "GAIN"
- board text added: "GND"
- board text added: "GVDD"
- board text added: "L TRIM"
- board text added: "LIN"
- board text added: "MUTE"
- board text added: "PLIM"
- board text added: "R TRIM"
- board text added: "RIN"
- board text added: "SYNC"
- board text added: "VCC"

Commit message: bak
Parts:
- added G***: LOGO, HammerheadAudio:Screamer_6x9mm, B.Cu at (122.0, 90.0)
- added G***: LOGO, HammerheadAudio:Screamer_6x9mm, F.Cu at (122.0, 90.0)
- added G***: LOGO, HammerheadAudio:Screamer_6x9mm, F.Cu at (122.0, 40.0)
- added G***: LOGO, HammerheadAudio:Screamer_6x9mm, B.Cu at (122.0, 40.0)
- added REF**: JLC_ToolingHole, HammerheadAudio:JLC_ToolingHole, F.Cu at (66.0, 94.0)
- added REF**: JLC_ToolingHole, HammerheadAudio:JLC_ToolingHole, F.Cu at (66.0, 36.0)
- added REF**: JLC_ToolingHole, HammerheadAudio:JLC_ToolingHole, F.Cu at (144.0, 36.0)
- added REF**: JLC_ToolingHole, HammerheadAudio:JLC_ToolingHole, F.Cu at (144.0, 94.0)
- moved J1 0.25 mm to (73.0, 65.0)
Routing:
- net VCC: track 317.9 -> 375.3 mm
- net GND: track 71.4 -> 76.1 mm, vias 145 -> 137
Other:
- board text added: "CLASS D AMPLIFIER V0.1 - FEB 2022 E. PALAIMA - HAMMERHEAD AUDIO"
- board text added: "JLCJLCJLCJLC"
- board text added: "L+"
- board text added: "LEFT"
- board text added: "LR IN"
- board text added: "PWR"
- board text added: "R+"

Commit message: schematic
Parts:
- removed G*** (x4): LOGO, HammerheadAudio:Screamer_6x9mm
- removed J12: PLIM_DEF, Connector_PinHeader_2.54mm:PinHeader_1x02_P2.54mm_Vertical_SMD_Pin1Right
- removed J4: ST/MN, Connector_PinHeader_2.54mm:PinHeader_2x03_P2.54mm_Vertical_SMD
- removed J5: GAIN_DEF, Connector_PinHeader_2.54mm:PinHeader_1x02_P2.54mm_Vertical_SMD_Pin1Right
- removed JP1: PWR, Jumper:SolderJumper-2_P1.3mm_Open_Pad1.0x1.5mm
- removed JP2: GND, Jumper:SolderJumper-2_P1.3mm_Open_Pad1.0x1.5mm
- removed JP3: R+, Jumper:SolderJumper-2_P1.3mm_Open_Pad1.0x1.5mm
- removed JP4: L+, Jumper:SolderJumper-2_P1.3mm_Open_Pad1.0x1.5mm
- removed R10: 5.6k, Resistor_SMD:R_0603_1608Metric_Pad1.05x0.95mm_HandSolder_SmallRef
- removed REF** (x4): JLC_ToolingHole, HammerheadAudio:JLC_ToolingHole
- added R18: 100k, Resistor_SMD:R_0603_1608Metric_Pad1.05x0.95mm_HandSolder_SmallRef, F.Cu at (48.8, 51.3)
- added R19: 20k, Resistor_SMD:R_0603_1608Metric_Pad1.05x0.95mm_HandSolder_SmallRef, F.Cu at (48.8, 53.8)
- added R20: 100k, Resistor_SMD:R_0603_1608Metric_Pad1.05x0.95mm_HandSolder_SmallRef, F.Cu at (53.2, 48.8)
- added R21: 39k, Resistor_SMD:R_0603_1608Metric_Pad1.05x0.95mm_HandSolder_SmallRef, F.Cu at (40.3, 65.7)
- added R22: 75k, Resistor_SMD:R_0603_1608Metric_Pad1.05x0.95mm_HandSolder_SmallRef, F.Cu at (53.2, 51.3)
- added R23: 47k, Resistor_SMD:R_0603_1608Metric_Pad1.05x0.95mm_HandSolder_SmallRef, F.Cu at (48.8, 56.3)
- added R24: 51k, Resistor_SMD:R_0603_1608Metric_Pad1.05x0.95mm_HandSolder_SmallRef, F.Cu at (36.0, 68.2)
- added R25: 51k, Resistor_SMD:R_0603_1608Metric_Pad1.05x0.95mm_HandSolder_SmallRef, F.Cu at (53.2, 53.8)
- added R26: 47k, Resistor_SMD:R_0603_1608Metric_Pad1.05x0.95mm_HandSolder_SmallRef, F.Cu at (57.5, 48.8)
- added R27: 75k, Resistor_SMD:R_0603_1608Metric_Pad1.05x0.95mm_HandSolder_SmallRef, F.Cu at (40.3, 68.2)
- added R28: 39k, Resistor_SMD:R_0603_1608Metric_Pad1.05x0.95mm_HandSolder_SmallRef, F.Cu at (48.8, 58.8)
- added R29: 100k, Resistor_SMD:R_0603_1608Metric_Pad1.05x0.95mm_HandSolder_SmallRef, F.Cu at (44.7, 65.7)
- added R30: 16k, Resistor_SMD:R_0603_1608Metric_Pad1.05x0.95mm_HandSolder_SmallRef, F.Cu at (48.8, 61.3)
- added R31: 100k, Resistor_SMD:R_0603_1608Metric_Pad1.05x0.95mm_HandSolder_SmallRef, F.Cu at (57.5, 51.3)
- added R32: 10k, Resistor_SMD:R_0603_1608Metric_Pad1.05x0.95mm_HandSolder_SmallRef, F.Cu at (53.2, 56.3)
- C10: value 47pf -> 1nf
- J6: value SYNC_DEFAULT -> GAIN_SEL; footprint Connector_PinHeader_2.54mm:PinHeader_1x02_P2.54mm_Vertical_SMD_Pin1Right -> Connector_PinHeader_2.54mm:PinHeader_2x08_P2.54mm_Vertical_SMD
- J7: value MN -> SYNC; footprint Connector_PinHeader_2.54mm:PinHeader_1x02_P2.54mm_Vertical_SMD_Pin1Right -> Connector_PinHeader_2.54mm:PinHeader_2x03_P2.54mm_Vertical_SMD
- J8: value MN -> PLIM_SEL; footprint Connector_PinHeader_2.54mm:PinHeader_1x02_P2.54mm_Vertical_SMD_Pin1Right -> Connector_PinHeader_2.54mm:PinHeader_2x02_P2.54mm_Vertical_SMD
- R15: value 4.7k -> 5.6k
- moved J8 83.1 mm to (40.2, 60.8), turned to 0 degrees
- moved J7 82.1 mm to (40.2, 52.4), turned to 0 degrees
- moved J6 78.6 mm to (27.4, 58.7)
- moved R15 73.0 mm to (36.0, 65.7), turned to 0 degrees
- moved C10 69.5 mm to (48.8, 48.8), turned to 0 degrees
Connections:
- C10 pad 1: Net-(C10-Pad1) -> GND
- C10 pad 2: GND -> Net-(C10-Pad2)
- C5 pad 1: Net-(C5-Pad1) -> LIN+
- C6 pad 1: Net-(C6-Pad1) -> LIN-
- J10 pad 1: L+ -> XOUT-
- J10 pad 2: R+ -> XOUT+
- J13 pad 13: L- -> Net-(J13-Pad13)
- J13 pad 2: R+ -> Net-(J13-Pad2)
- J13 pad 7: R- -> XOUT+
- J13 pad 8: L+ -> XOUT-
- J2 pad 3: (no net) -> Net-(J2-Pad3)
- J6 pad 1: SYNC -> M20DB
- J6 pad 2: Net-(J6-Pad2) -> GAIN
- J7 pad 1: Net-(C16-Pad2) -> Net-(J7-Pad1)
- J7 pad 2: Net-(C14-Pad1) -> Net-(J7-Pad2)
- J8 pad 1: Net-(C17-Pad2) -> GVDD
- J8 pad 2: Net-(C15-Pad1) -> PLIM
- R15 pad 1: Net-(C10-Pad1) -> GND
- R15 pad 2: Net-(J6-Pad2) -> M20DB
- U3 pad 16: SYNC -> Net-(J7-Pad1)
Routing:
- net L+: track 133.7 -> 12.9 mm
- net R+: track 117.8 -> 0.00 mm
- net L-: track 51.1 -> 0.00 mm
- net R-: track 98.7 -> 55.3 mm
- net GVDD: track 37.4 -> 0.00 mm, vias 1 -> 0
- net GAIN: track 30.7 -> 0.00 mm, vias 1 -> 0
- net Net-(C6-Pad1): track 17.1 -> 0.00 mm
- net LIN-: track 12.3 -> 29.4 mm
- net XOUT+: track 0.00 -> 8.02 mm
- net XOUT-: track 0.00 -> 8.01 mm
- net Net-(C5-Pad1): track 7.79 -> 0.00 mm
- net LIN+: track 17.8 -> 25.6 mm
- net Net-(J6-Pad2): track 6.51 -> 0.00 mm
- net Net-(J16-Pad1): track 5.45 -> 0.00 mm
- net Net-(J15-Pad1): track 5.45 -> 0.00 mm
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Other:
- board text added: "XOUT"
- board text removed: "STEREO"
- board text removed: "SYNC DEFAULT"

Commit message: layout progress
Parts:
- moved R15 76.1 mm to (109.7, 47.0), turned to 180 degrees
- moved R24 74.0 mm to (109.7, 74.0), turned to 180 degrees
- moved J6 73.8 mm to (100.9, 65.9)
- moved R21 70.7 mm to (109.7, 52.3), turned to 180 degrees
- moved R27 69.8 mm to (109.7, 75.8), turned to 180 degrees
- moved J7 67.8 mm to (100.8, 82.8)
- moved C10 66.6 mm to (102.5, 88.1)
- moved R29 66.5 mm to (109.7, 79.4), turned to 180 degrees
- moved R30 65.3 mm to (109.7, 84.7), turned to 180 degrees
- moved R28 64.9 mm to (109.7, 81.2), turned to 180 degrees
- moved J8 61.5 mm to (100.8, 50.3)
- moved R19 61.1 mm to (109.7, 48.8), turned to 180 degrees
- moved R31 61.1 mm to (109.7, 82.9), turned to 180 degrees
- moved R18 60.9 mm to (109.7, 50.5), turned to 180 degrees
- moved R23 60.9 mm to (109.7, 55.9), turned to 180 degrees
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Routing:
- net R+: track 0.00 -> 50.7 mm
- net L-: track 0.00 -> 50.4 mm
- net SYNC: track 44.0 -> 0.00 mm
- net L+: track 12.9 -> 52.6 mm
- net PLIM: track 37.7 -> 0.00 mm, vias 1 -> 0
- net RIN: track 35.8 -> 0.00 mm
- net FAULT: track 34.8 -> 0.00 mm, vias 1 -> 0
- net LIN-: track 29.4 -> 0.00 mm
- net Net-(C15-Pad1): track 48.3 -> 19.1 mm
- net Net-(C16-Pad2): track 36.5 -> 9.13 mm
- net LIN+: track 25.6 -> 0.00 mm
- net Net-(Q4-Pad3): track 35.6 -> 11.1 mm
- net RIN-: track 21.5 -> 0.00 mm
- net Net-(C14-Pad1): track 34.8 -> 14.6 mm
- net RIN+: track 19.3 -> 0.00 mm
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Other:
- board text added: "DFLT"
- board text added: "EXT"
- board text added: "FLT"
- board text added: "GAIN_SEL"
- board text added: "M20"
- board text added: "M26"
- board text added: "M32"
- board text added: "M36"
- board text added: "S20"
- board text added: "S26"
- board text added: "S32"
- board text added: "S36"
- board text added: "SYNC_MODE"
- board text removed: "GAIN DEFAULT"
- board text removed: "MONO"
- board text removed: "PLIM DEFAULT"
- board text removed: "STEREO VS MONO"
