File: AmpClassD_Daugher.kicad_pcb (KiCad board)
At the start: 2 copper layers, 80 x 60 mm, 88 parts, among them J1 POWER, J10 MONO, J11 LEFT, J13 OUTS, J14 INS, J15 PWR, J16 GND, J17 R+, J18 L+, J2 POWER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

Commit message: update finished
Parts:
- added G***: LOGO, HammerheadAudio:Screamer_6x9mm, B.Cu at (127.5, 40.0)
- added G***: LOGO, HammerheadAudio:Screamer_6x9mm, B.Cu at (127.5, 90.0)
- added G***: LOGO, HammerheadAudio:Screamer_6x9mm, F.Cu at (127.5, 90.0)
- added G***: LOGO, HammerheadAudio:Screamer_6x9mm, F.Cu at (127.5, 40.0)
- added REF**: JLC_ToolingHole, HammerheadAudio:JLC_ToolingHole, F.Cu at (144.0, 94.0)
- added REF**: JLC_ToolingHole, HammerheadAudio:JLC_ToolingHole, F.Cu at (66.0, 94.0)
- added REF**: JLC_ToolingHole, HammerheadAudio:JLC_ToolingHole, F.Cu at (66.0, 36.0)
- added REF**: JLC_ToolingHole, HammerheadAudio:JLC_ToolingHole, F.Cu at (144.0, 36.0)
- moved R32 5.33 mm to (103.4, 88.1), turned to 0 degrees
- moved C10 4.25 mm to (98.2, 88.1)
- moved R24 0.89 mm to (108.9, 74.0)
- moved R25 0.89 mm to (108.8, 72.3)
- moved R26 0.89 mm to (108.8, 77.6)
- moved R27 0.89 mm to (108.8, 75.8)
- moved R28 0.89 mm to (108.8, 81.2)
- moved R29 0.89 mm to (108.8, 79.4)
- moved R30 0.89 mm to (108.8, 84.7)
- moved R31 0.89 mm to (108.8, 82.9)
- moved R15 0.83 mm to (108.9, 47.0)
- moved R18 0.83 mm to (108.9, 50.5)
- moved R19 0.83 mm to (108.9, 48.8)
- moved R20 0.83 mm to (108.9, 54.1)
- moved R21 0.83 mm to (108.9, 52.3)
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Connections:
- J6 pad 1: M20DB -> GAIN
- J6 pad 10: GAIN -> S20DB
- J6 pad 11: S26DB -> GAIN
- J6 pad 12: GAIN -> S26DB
- J6 pad 13: S32DB -> GAIN
- J6 pad 14: GAIN -> S32DB
- J6 pad 15: S36DB -> GAIN
- J6 pad 16: GAIN -> S36DB
- J6 pad 2: GAIN -> M20DB
- J6 pad 3: M26DB -> GAIN
- J6 pad 4: GAIN -> M26DB
- J6 pad 5: M32DB -> GAIN
- J6 pad 6: GAIN -> M32DB
- J6 pad 7: M36DB -> GAIN
- J6 pad 8: GAIN -> M36DB
- J6 pad 9: S20DB -> GAIN
- J7 pad 3: Net-(J7-Pad1) -> SYNC
- J7 pad 4: SYNC -> Net-(J7-Pad2)
- J7 pad 5: Net-(J7-Pad1) -> Net-(C10-Pad2)
- J7 pad 6: Net-(C10-Pad2) -> Net-(J7-Pad2)
- R32 pad 2: Net-(J7-Pad2) -> Net-(J7-Pad1)
- U3 pad 16: Net-(J7-Pad1) -> Net-(J7-Pad2)
Routing:
- net GVDD: track 0.00 -> 98.8 mm, vias 0 -> 4
- net GAIN: track 0.00 -> 73.5 mm, vias 0 -> 4
- net Net-(Q4-Pad3): track 11.1 -> 69.5 mm
- net PLIM: track 0.00 -> 52.4 mm, vias 0 -> 1
- net FAULT: track 0.00 -> 37.6 mm, vias 0 -> 1
- net RIN: track 0.00 -> 34.4 mm
- net Net-(J7-Pad2): track 0.00 -> 34.0 mm
- net VCC: track 368.3 -> 398.4 mm, vias 0 -> 2
- net GND: track 67.4 -> 97.5 mm, vias 84 -> 103
- net SYNC: track 0.00 -> 29.2 mm
- net LIN-: track 0.00 -> 28.6 mm
- net LIN+: track 0.00 -> 24.7 mm
- net Net-(R14-Pad1): track 4.24 -> 25.9 mm
- net RIN+: track 0.00 -> 16.9 mm
- net RIN-: track 0.00 -> 16.8 mm
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Other:
- board text added: "CAP"
- board text added: "CLASS D AMPLIFIER V1.1 - JULY 2023 E. PALAIMA - HAMMERHEAD AUDIO JLCJLCJLCJLC"
- board text added: "M_OUT"
- board text added: "S_IN"
- board text added: "| L+ |"
- board text added: "| L- |"
- board text added: "| R+ |"
- board text added: "| R- |"
- board text removed: "CLASS D AMPLIFIER V0.1 - FEB 2022 E. PALAIMA - HAMMERHEAD AUDIO"
- board text removed: "FLT"
- board text removed: "JLCJLCJLCJLC"
- board text removed: "L+"
- board text removed: "R+"
- board text removed: "| L- | L+ | R- | R+ |"
