File: AmpClassD_Daugher.sch (KiCad schematic (older format))
At the start: 67 parts, among them J1 POWER, J10 MONO, J11 LEFT, J2 POWER, J3 AUDIO_IN, J4 ST/MN, J5 GAIN_DEFAULT, J6 SYNC_DEFAULT, J7 MN, J8 MN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

Commit message: schematic updates
Parts:
- added D2: M7, Diode_SMD:D_SMA, symbol Device:D
- added J12: INS, Connector_PinHeader_2.54mm:PinHeader_1x14_P2.54mm_Vertical, symbol Connector:Conn_01x14_Male
- added J13: OUTS, Connector_PinHeader_2.54mm:PinHeader_1x14_P2.54mm_Vertical, symbol Connector:Conn_01x14_Male
- added J14: PLIM_DEF, Connector_PinHeader_2.54mm:PinHeader_1x02_P2.54mm_Vertical_SMD_Pin1Right, symbol Connector:Conn_01x02_Male
- added Q5: MMBT3904, Package_TO_SOT_SMD:SOT-23, symbol Transistor_BJT:MMBT3904
- added R17: 100k, Resistor_SMD:R_0603_1608Metric_Pad1.05x0.95mm_HandSolder_SmallRef, symbol Device:R
- J5: value GAIN_DEFAULT -> GAIN_DEF
- RV1, RV2: value 2.2k -> 20k
Connections:
- net labels added: FAULT, PLIM
- net labels removed: +24V
- wire segments 271 -> 325
Other:
- moved on the sheet: C11, D1, J3, Q1, Q3, R12, R9

Commit message: layout progress
Parts:
- added J15: PWR, HammerheadAudio:M3_Plated, symbol Connector:Conn_01x01_Female
- added J16: GND, HammerheadAudio:M3_Plated, symbol Connector:Conn_01x01_Female
- added J17: R+, HammerheadAudio:M3_Plated, symbol Connector:Conn_01x01_Female
- added J18: L+, HammerheadAudio:M3_Plated, symbol Connector:Conn_01x01_Female
- added JP1: PWR, Jumper:SolderJumper-2_P1.3mm_Open_Pad1.0x1.5mm, symbol Device:Jumper_NO_Small
- added JP2: GND, Jumper:SolderJumper-2_P1.3mm_Open_Pad1.0x1.5mm, symbol Device:Jumper_NO_Small
- added JP3: R+, Jumper:SolderJumper-2_P1.3mm_Open_Pad1.0x1.5mm, symbol Device:Jumper_NO_Small
- added JP4: L+, Jumper:SolderJumper-2_P1.3mm_Open_Pad1.0x1.5mm, symbol Device:Jumper_NO_Small
- J1, J10, J11, J9: footprint HammerheadAudio:Phoenix_Stacked_Marking2_Wider_NoRef -> HammerheadAudio:Phoenix_Stacked_Marking2_Wider_NoRef_Centered
Connections:
- net GND: now also JP2.2
- net L+: now also JP4.2
- net R+: now also J13.2 (Pin_2), J13.3 (Pin_3), J13.4 (Pin_4), JP3.2; no longer J13.5 (Pin_5), J13.6 (Pin_6), J13.7 (Pin_7)
- net R-: now also J13.5 (Pin_5), J13.6 (Pin_6), J13.7 (Pin_7); no longer J13.2 (Pin_2), J13.3 (Pin_3), J13.4 (Pin_4)
- net VCC: now also JP1.2
- new net: J15.1 (Pin_1), JP1.1
- new net: J16.1 (Pin_1), JP2.1
- new net: J17.1 (Pin_1), JP3.1
- new net: J18.1 (Pin_1), JP4.1
Changed lines of the file:
@@
 F 0 "J9" H 10668 2375 50  0000 C CNN
 F 1 "RIGHT" H 10668 2466 50  0000 C CNN
-F 2 "HammerheadAudio:Phoenix_Stacked_Marking2_Wider_NoRef" H 10750 2700 50  0001 C CNN
+F 2 "HammerheadAudio:Phoenix_Stacked_Marking2_Wider_NoRef_Centered" H 10750 2700 50  0001 C CNN
 F 3 "~" H 10750 2700 50  0001 C CNN
 	1    10750 2700
@@
 F 0 "J10" H 10668 2925 50  0000 C CNN
 F 1 "MONO" H 10668 3016 50  0000 C CNN
-F 2 "HammerheadAudio:Phoenix_Stacked_Marking2_Wider_NoRef" H 10750 3250 50  0001 C CNN
+F 2 "HammerheadAudio:Phoenix_Stacked_Marking2_Wider_NoRef_Centered" H 10750 3250 50  0001 C CNN
 F 3 "~" H 10750 3250 50  0001 C CNN
 	1    10750 3250
@@
 F 0 "J11" H 10668 3475 50  0000 C CNN
 F 1 "LEFT" H 10668 3566 50  0000 C CNN
-F 2 "HammerheadAudio:Phoenix_Stacked_Marking2_Wider_NoRef" H 10750 3800 50  0001 C CNN
+F 2 "HammerheadAudio:Phoenix_Stacked_Marking2_Wider_NoRef_Centered" H 10750 3800 50  0001 C CNN
 F 3 "~" H 10750 3800 50  0001 C CNN
 	1    10750 3800
@@
 F 0 "J1" H 618 675 50  0000 C CNN
 F 1 "POWER" H 618 766 50  0000 C CNN
-F 2 "HammerheadAudio:Phoenix_Stacked_Marking2_Wider_NoRef" H 700 1000 50  0001 C CNN
+F 2 "HammerheadAudio:Phoenix_Stacked_Marking2_Wider_NoRef_Centered" H 700 1000 50  0001 C CNN
 F 3 "~" H 700 1000 50  0001 C CNN
 	1    700  1000
@@
 	1    0    0    -1
 $EndComp
-Text GLabel 2550 3250 2    50   Input ~ 0
+Text GLabel 2550 3550 2    50   Input ~ 0
 R-
 Text GLabel 2550 3850 2    50   Input ~ 0
@@
 Text GLabel 2550 3750 2    50   Input ~ 0
 L+
-Text GLabel 2550 3650 2    50   Input ~ 0
+Text GLabel 2550 3350 2    50   Input ~ 0
 R+
 Wire Wire Line
@@
 Wire Wire Line
 	1450 3150 1400 3150
-Text GLabel 2550 3550 2    50   Input ~ 0
+Text GLabel 2550 3250 2    50   Input ~ 0
 R+
 Wire Wire Line
@@
 Wire Wire Line
 	2450 3550 2550 3550
-Text GLabel 2550 3350 2    50   Input ~ 0
+Text GLabel 2550 3650 2    50   Input ~ 0
 R-
 Wire Wire Line
@@
 Wire Wire Line
 	1450 4150 1600 4150
+Text GLabel 2550 3450 2    50   Input ~ 0
+R-
+Wire Wire Line
+	2450 3150 2550 3150
 Text GLabel 2550 3150 2    50   Input ~ 0
-R-
-Wire Wire Line
-	2450 3150 2550 3150
-Text GLabel 2550 3450 2    50   Input ~ 0
 R+
 Wire Wire Line
@@
 Wire Wire Line
 	2450 4350 2700 4350
+$Comp
+L Connector:Conn_01x01_Female J15
+U 1 1 6354D0B7
+P 7100 6900
+F 0 "J15" H 6992 6675 50  0000 C CNN
+F 1 "PWR" H 6992 6766 50  0000 C CNN
+F 2 "HammerheadAudio:M3_Plated" H 7100 6900 50  0001 C CNN
+F 3 "~" H 7100 6900 50  0001 C CNN
+	1    7100 6900
+	-1   0    0    1
+$EndComp
+$Comp
+L Connector:Conn_01x01_Female J16
+U 1 1 635549EB
+P 7900 6900
+F 0 "J16" H 7792 6675 50  0000 C CNN
+F 1 "GND" H 7792 6766 50  0000 C CNN
+F 2 "HammerheadAudio:M3_Plated" H 7900 6900 50  0001 C CNN
+F 3 "~" H 7900 6900 50  0001 C CNN
+	1    7900 6900
+	-1   0    0    1
+$EndComp
+$Comp
+L Device:Jumper_NO_Small JP1
+U 1 1 635554C5
+P 7450 6900
+F 0 "JP1" H 7450 7085 50  0000 C CNN
+F 1 "PWR" H 7450 6994 50  0000 C CNN
+F 2 "Jumper:SolderJumper-2_P1.3mm_Open_Pad1.0x1.5mm" H 7450 6900 50  0001 C CNN
+F 3 "~" H 7450 6900 50  0001 C CNN
+	1    7450 6900
+	1    0    0    -1
+$EndComp
+Wire Wire Line
+	7300 6900 7350 6900
+$Comp
+L power:VCC #PWR035
+U 1 1 63577A57
+P 7600 6900
+F 0 "#PWR035" H 7600 6750 50  0001 C CNN
+F 1 "VCC" H 7617 7073 50  0000 C CNN
+F 2 "" H 7600 6900 50  0001 C CNN
+F 3 "" H 7600 6900 50  0001 C CNN
+	1    7600 6900
+	0    1    1    0
+$EndComp
+Wire Wire Line
+	7550 6900 7600 6900
+$Comp
+L Device:Jumper_NO_Small JP2
+U 1 1 63599BCE
+P 8250 6900
+F 0 "JP2" H 8250 7085 50  0000 C CNN
+F 1 "GND" H 8250 6994 50  0000 C CNN
+F 2 "Jumper:SolderJumper-2_P1.3mm_Open_Pad1.0x1.5mm" H 8250 6900 50  0001 C CNN
+F 3 "~" H 8250 6900 50  0001 C CNN
+	1    8250 6900
+	1    0    0    -1
+$EndComp
+Wire Wire Line
+	8100 6900 8150 6900
+Wire Wire Line
+	8350 6900 8400 6900
+$Comp
+L power:GND #PWR036
+U 1 1 635BBA28
+P 8400 6900
+F 0 "#PWR036" H 8400 6650 50  0001 C CNN
+F 1 "GND" H 8405 6727 50  0000 C CNN
+F 2 "" H 8400 6900 50  0001 C CNN
+F 3 "" H 8400 6900 50  0001 C CNN
+	1    8400 6900
+	0    -1   -1   0
+$EndComp
+$Comp
+L Connector:Conn_01x01_Female J17
+U 1 1 635BC077
+P 8700 6900
+F 0 "J17" H 8592 6675 50  0000 C CNN
+F 1 "R+" H 8592 6766 50  0000 C CNN
+F 2 "HammerheadAudio:M3_Plated" H 8700 6900 50  0001 C CNN
+F 3 "~" H 8700 6900 50  0001 C CNN
+	1    8700 6900
+	-1   0    0    1
+$EndComp
+$Comp
+L Connector:Conn_01x01_Female J18
+U 1 1 635BC081
+P 9650 6900
+F 0 "J18" H 9542 6675 50  0000 C CNN
+F 1 "L+" H 9542 6766 50  0000 C CNN
+F 2 "HammerheadAudio:M3_Plated" H 9650 6900 50  0001 C CNN
+F 3 "~" H 9650 6900 50  0001 C CNN
+	1    9650 6900
+	-1   0    0    1
+$EndComp
+$Comp
+L Device:Jumper_NO_Small JP3
+U 1 1 635BC08B
+P 9050 6900
+F 0 "JP3" H 9050 7085 50  0000 C CNN
+F 1 "R+" H 9050 6994 50  0000 C CNN
+F 2 "Jumper:SolderJumper-2_P1.3mm_Open_Pad1.0x1.5mm" H 9050 6900 50  0001 C CNN
+F 3 "~" H 9050 6900 50  0001 C CNN
+	1    9050 6900
+	1    0    0    -1
+$EndComp
+Wire Wire Line
+	8900 6900 8950 6900
+Wire Wire Line
+	9150 6900 9200 6900
+$Comp
+L Device:Jumper_NO_Small JP4
+U 1 1 635BC0A1
+P 10000 6900
+F 0 "JP4" H 10000 7085 50  0000 C CNN
+F 1 "L+" H 10000 6994 50  0000 C CNN
+F 2 "Jumper:SolderJumper-2_P1.3mm_Open_Pad1.0x1.5mm" H 10000 6900 50  0001 C CNN
+F 3 "~" H 10000 6900 50  0001 C CNN
+	1    10000 6900
+	1    0    0    -1
+$EndComp
+Wire Wire Line
+	9850 6900 9900 6900
+Wire Wire Line
+	10100 6900 10150 6900
+Text GLabel 10150 6900 2    50   Input ~ 0
+L+
+Text GLabel 9200 6900 2    50   Input ~ 0
+R+
 $EndSCHEMATC

Commit message: layout progress
Parts:
- renumbered J14 to J12, J12 to J14
Changed lines of the file:
@@
 $EndComp
 $Comp
-L Connector:Conn_01x14_Male J12
+L Connector:Conn_01x14_Male J14
 U 1 1 62B05122
 P 1800 3650
-F 0 "J12" H 1772 3624 50  0000 R CNN
+F 0 "J14" H 1772 3624 50  0000 R CNN
 F 1 "INS" H 1772 3533 50  0000 R CNN
 F 2 "Connector_PinHeader_2.54mm:PinHeader_1x14_P2.54mm_Vertical" H 1800 3650 50  0001 C CNN
@@
 	2250 1600 2550 1600
 $Comp
-L Connector:Conn_01x02_Male J14
+L Connector:Conn_01x02_Male J12
 U 1 1 630F5309
 P 6300 3350
-F 0 "J14" H 6272 3232 50  0000 R CNN
+F 0 "J12" H 6272 3232 50  0000 R CNN
 F 1 "PLIM_DEF" H 6272 3323 50  0000 R CNN
 F 2 "Connector_PinHeader_2.54mm:PinHeader_1x02_P2.54mm_Vertical_SMD_Pin1Right" H 6300 3350 50  0001 C CNN

Commit message: layout progress
Parts:
- J3: symbol Crossley_Symbols:TRS_BalancedJack -> Connector:AudioJack3
Connections:
- net GND: now also J3.S; no longer J3.1 (S)
- net LIN: now also J3.T; no longer J3.2 (T)
- net LIN+: now also J4.3 (Pin_3); no longer J4.4 (Pin_4)
- net LIN-: now also J4.4 (Pin_4); no longer J4.3 (Pin_3)
- net RIN: now also J3.R; no longer J3.3 (R)
- net at C5.1: now also J4.1 (Pin_1); no longer J4.2 (Pin_2)
- net at C6.1: now also J4.2 (Pin_2); no longer J4.1 (Pin_1)
Changed lines of the file:
@@
 L Connector_Generic:Conn_02x03_Odd_Even J4
 U 1 1 633BE700
-P 4200 6950
-F 0 "J4" V 4296 6762 50  0000 R CNN
-F 1 "ST/MN" V 4205 6762 50  0000 R CNN
-F 2 "Connector_PinHeader_2.54mm:PinHeader_2x03_P2.54mm_Vertical_SMD" H 4200 6950 50  0001 C CNN
-F 3 "C192301" H 4200 6950 50  0001 C CNN
-	1    4200 6950
-	0    -1   -1   0
+P 4200 6850
+F 0 "J4" V 4296 6662 50  0000 R CNN
+F 1 "ST/MN" V 4205 6662 50  0000 R CNN
+F 2 "Connector_PinHeader_2.54mm:PinHeader_2x03_P2.54mm_Vertical_SMD" H 4200 6850 50  0001 C CNN
+F 3 "C192301" H 4200 6850 50  0001 C CNN
+	1    4200 6850
+	0    -1   1    0
 $EndComp
 Wire Wire Line
@@
 	5350 3650 6600 3650
 $Comp
-L Crossley_Symbols:TRS_BalancedJack J3
+L Connector:AudioJack3 J3
 U 1 1 61CD5AC7
 P 3750 1250

Commit message: updated schematic
Parts:
- removed J12: PLIM_DEF, Connector_PinHeader_2.54mm:PinHeader_1x02_P2.54mm_Vertical_SMD_Pin1Right, symbol Connector:Conn_01x02_Male
- removed J6: SYNC_DEFAULT, Connector_PinHeader_2.54mm:PinHeader_1x02_P2.54mm_Vertical_SMD_Pin1Right, symbol Connector:Conn_01x02_Male
- removed J7, J8: MN, Connector_PinHeader_2.54mm:PinHeader_1x02_P2.54mm_Vertical_SMD_Pin1Right, symbol Connector:Conn_01x02_Male
- added J6: Conn_02x08_Odd_Even, symbol Connector_Generic:Conn_02x08_Odd_Even
- added J7: ST/MN, Connector_PinHeader_2.54mm:PinHeader_2x03_P2.54mm_Vertical_SMD, symbol Connector_Generic:Conn_02x03_Odd_Even
- added J8: PLIM_SEL, symbol Connector_Generic:Conn_02x02_Odd_Even
- added R18, R20, R29, R31: 100k, Resistor_SMD:R_0603_1608Metric_Pad1.05x0.95mm_HandSolder_SmallRef, symbol Device:R
- added R19: 20k, Resistor_SMD:R_0603_1608Metric_Pad1.05x0.95mm_HandSolder_SmallRef, symbol Device:R
- added R21, R28: 39k, Resistor_SMD:R_0603_1608Metric_Pad1.05x0.95mm_HandSolder_SmallRef, symbol Device:R
- added R22, R27: 75k, Resistor_SMD:R_0603_1608Metric_Pad1.05x0.95mm_HandSolder_SmallRef, symbol Device:R
- added R23, R26: 47k, Resistor_SMD:R_0603_1608Metric_Pad1.05x0.95mm_HandSolder_SmallRef, symbol Device:R
- added R24, R25: 51k, Resistor_SMD:R_0603_1608Metric_Pad1.05x0.95mm_HandSolder_SmallRef, symbol Device:R
- added R30: 16k, Resistor_SMD:R_0603_1608Metric_Pad1.05x0.95mm_HandSolder_SmallRef, symbol Device:R
- added R32: 10k, Resistor_SMD:R_0603_1608Metric_Pad1.05x0.95mm_HandSolder_SmallRef, symbol Device:R
- C10: value 47pf -> 1nf
- R15: value 4.7k -> 5.6k
Connections:
- net GAIN: now also J6.10 (Pin_10), J6.12 (Pin_12), J6.14 (Pin_14), J6.16 (Pin_16), J6.2 (Pin_2), J6.4 (Pin_4), J6.6 (Pin_6), J6.8 (Pin_8)
- net GND: now also C10.1, R15.1, R19.1, R21.1, R23.1, R25.1, R27.1, R29.1, R31.1; no longer C10.2
- net GVDD: now also J8.1 (Pin_1), R18.1, R20.1, R22.1, R24.1, R26.1, R28.1, R30.1
- net L+: no longer J10.1 (Pin_1), J13.8 (Pin_8)
- net PLIM: now also J8.2 (Pin_2), J8.4 (Pin_4)
- net R+: no longer J10.2 (Pin_2)
- net R-: no longer J13.7 (Pin_7)
- net SYNC: now also J7.4 (Pin_4), R32.1; no longer U3.16 (SYNC)
- net M20DB: now reaches R15.2
- net M20DB: now also J6.1 (Pin_1)
- new net: J7.1 (Pin_1), J7.3 (Pin_3), J7.5 (Pin_5), U3.16 (SYNC)
- new net: J7.2 (Pin_2), R32.2
- new net: C10.2, J7.6 (Pin_6)
- new net M26DB: J6.3 (Pin_3), R18.2, R19.2
- new net M32DB: J6.5 (Pin_5), R20.2, R21.2
- new net M36DB: J6.7 (Pin_7), R22.2, R23.2
- new net S20DB: J6.9 (Pin_9), R24.2, R25.2
- new net S26DB: J6.11 (Pin_11), R26.2, R27.2
- new net S32DB: J6.13 (Pin_13), R28.2, R29.2
- new net S36DB: J6.15 (Pin_15), R30.2, R31.2
- new net XOUT+: J10.2 (Pin_2), J13.7 (Pin_7)
- new net XOUT-: J10.1 (Pin_1), J13.8 (Pin_8)
- no-connect marks 1 -> 2

Commit message: schematic
Parts:
- removed J4: ST/MN, Connector_PinHeader_2.54mm:PinHeader_2x03_P2.54mm_Vertical_SMD, symbol Connector_Generic:Conn_02x03_Odd_Even
- removed J5: GAIN_DEF, Connector_PinHeader_2.54mm:PinHeader_1x02_P2.54mm_Vertical_SMD_Pin1Right, symbol Connector:Conn_01x02_Male
- removed JP1: PWR, Jumper:SolderJumper-2_P1.3mm_Open_Pad1.0x1.5mm, symbol Device:Jumper_NO_Small
- removed JP2: GND, Jumper:SolderJumper-2_P1.3mm_Open_Pad1.0x1.5mm, symbol Device:Jumper_NO_Small
- removed JP3: R+, Jumper:SolderJumper-2_P1.3mm_Open_Pad1.0x1.5mm, symbol Device:Jumper_NO_Small
- removed JP4: L+, Jumper:SolderJumper-2_P1.3mm_Open_Pad1.0x1.5mm, symbol Device:Jumper_NO_Small
- removed R10: 5.6k, Resistor_SMD:R_0603_1608Metric_Pad1.05x0.95mm_HandSolder_SmallRef, symbol Device:R
- C1, C2, C3, C4, C5, C6, C7, C8: LCSC (none) -> C440198
- C10, C18, C19, C20, C21, C23, C24: LCSC (none) -> C1588
- C11: LCSC (none) -> C15849
- C12, C13, C26, C9: LCSC (none) -> C14663
- C14, C15, C16, C17: LCSC (none) -> C21120
- C22, C25: LCSC (none) -> C311622
- D1: LCSC (none) -> C84256
- D2: LCSC (none) -> C95872
- FB1, FB2, FB3, FB4: LCSC (none) -> C124704
- J2: LCSC (none) -> C397342
- J3: LCSC (none) -> C879743
- J6: value Conn_02x08_Odd_Even -> GAIN_SEL; footprint (none) -> Connector_PinHeader_2.54mm:PinHeader_2x08_P2.54mm_Vertical_SMD; LCSC (none) -> C2884017
- J7: value ST/MN -> SYNC; LCSC (none) -> C780054
- J8: footprint (none) -> Connector_PinHeader_2.54mm:PinHeader_2x02_P2.54mm_Vertical_SMD; LCSC (none) -> C3294460
- Q1, Q2, Q3, Q4, Q5: LCSC (none) -> C20526
- R1, R2, R3, R4, R5, R6: LCSC (none) -> C22935
- R11, R12, R13, R14, R17, R18, R20, R29, R31, R8: LCSC (none) -> C25803
- R15: LCSC (none) -> C23189
- R16, R32: LCSC (none) -> C25804
- R19: LCSC (none) -> C4184
- R21, R28: LCSC (none) -> C23153
- R22, R27: LCSC (none) -> C23242
- R23, R26: LCSC (none) -> C23162
- R24, R25: LCSC (none) -> C23196
- R30: LCSC (none) -> C22818
- R7: LCSC (none) -> C21190
- R9: LCSC (none) -> C4190
- RV1, RV2: LCSC (none) -> C128550
- U1, U2: LCSC (none) -> C7426
- U3: LCSC (none) -> C46497
Connections:
- net L-: no longer J13.13 (Pin_13)
- net LIN+: now also C5.1
- net LIN-: now also C6.1
- net R+: no longer J13.2 (Pin_2)
- no-connect marks 2 -> 9

Commit message: update finished
Connections:
- net GAIN: now also J6.1 (Pin_1), J6.11 (Pin_11), J6.13 (Pin_13), J6.15 (Pin_15), J6.3 (Pin_3), J6.5 (Pin_5), J6.7 (Pin_7), J6.9 (Pin_9); no longer J6.10 (Pin_10), J6.12 (Pin_12), J6.14 (Pin_14), J6.16 (Pin_16), J6.2 (Pin_2), J6.4 (Pin_4), J6.6 (Pin_6), J6.8 (Pin_8)
- net M20DB: now also J6.2 (Pin_2); no longer J6.1 (Pin_1)
- net M26DB: now also J6.4 (Pin_4); no longer J6.3 (Pin_3)
- net M32DB: now also J6.6 (Pin_6); no longer J6.5 (Pin_5)
- net M36DB: now also J6.8 (Pin_8); no longer J6.7 (Pin_7)
- net S20DB: now also J6.10 (Pin_10); no longer J6.9 (Pin_9)
- net S26DB: now also J6.12 (Pin_12); no longer J6.11 (Pin_11)
- net S32DB: now also J6.14 (Pin_14); no longer J6.13 (Pin_13)
- net S36DB: now also J6.16 (Pin_16); no longer J6.15 (Pin_15)
- net SYNC: now also J7.3 (Pin_3); no longer J7.4 (Pin_4)
- net at J7.2 (Pin_2): now also J7.4 (Pin_4), J7.6 (Pin_6), U3.16 (SYNC); no longer R32.2
- net at C10.2: now also J7.5 (Pin_5); no longer J7.6 (Pin_6)
- new net: J7.1 (Pin_1), R32.2
Changed lines of the file:
@@
 	9850 6900 9900 6900
-$Comp
-L Connector_Generic:Conn_02x08_Odd_Even J6
-U 1 1 64DA7895
-P 5100 -850
-F 0 "J6" H 5150 -333 50  0000 C CNN
-F 1 "GAIN_SEL" H 5150 -424 50  0000 C CNN
-F 2 "Connector_PinHeader_2.54mm:PinHeader_2x08_P2.54mm_Vertical_SMD" H 5100 -850 50  0001 C CNN
-F 3 "C2884017" H 5100 -850 50  0001 C CNN
-F 4 "C2884017" H 5100 -850 50  0001 C CNN "LCSC"
-	1    5100 -850
-	1    0    0    -1
-$EndComp
 $Comp
 L Device:R R15
@@
 L Connector_Generic:Conn_02x03_Odd_Even J7
 U 1 1 654D81DE
-P 6250 5800
-F 0 "J7" V 6346 5612 50  0000 R CNN
-F 1 "SYNC" V 6255 5612 50  0000 R CNN
-F 2 "Connector_PinHeader_2.54mm:PinHeader_2x03_P2.54mm_Vertical_SMD" H 6250 5800 50  0001 C CNN
-F 3 "C780054" H 6250 5800 50  0001 C CNN
-F 4 "C780054" H 6250 5800 50  0001 C CNN "LCSC"
-	1    6250 5800
-	-1   0    0    -1
+P 6150 5800
+F 0 "J7" V 6246 5612 50  0000 R CNN
+F 1 "SYNC" V 6155 5612 50  0000 R CNN
+F 2 "Connector_PinHeader_2.54mm:PinHeader_2x03_P2.54mm_Vertical_SMD" H 6150 5800 50  0001 C CNN
+F 3 "C780054" H 6150 5800 50  0001 C CNN
+F 4 "C780054" H 6150 5800 50  0001 C CNN "LCSC"
+	1    6150 5800
+	1    0    0    -1
 $EndComp
 $Comp
@@
 Wire Wire Line
 	3600 7000 3950 7000
+$Comp
+L Connector_Generic:Conn_02x08_Odd_Even J6
+U 1 1 64DA7895
+P 5200 -850
+F 0 "J6" H 5250 -333 50  0000 C CNN
+F 1 "GAIN_SEL" H 5250 -424 50  0000 C CNN
+F 2 "Connector_PinHeader_2.54mm:PinHeader_2x08_P2.54mm_Vertical_SMD" H 5200 -850 50  0001 C CNN
+F 3 "C2884017" H 5200 -850 50  0001 C CNN
+F 4 "C2884017" H 5200 -850 50  0001 C CNN "LCSC"
+	1    5200 -850
+	-1   0    0    -1
+$EndComp
 $EndSCHEMATC
